File: pcb/keyboard_pcb.kicad_sch (KiCad schematic)
At the start: 20 parts, among them J1 TRRS, K01 KEYSW, K02 KEYSW, K03 KEYSW, K04 KEYSW, K05 KEYSW, K11 KEYSW, K12 KEYSW, K13 KEYSW, K14 KEYSW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

Commit message: pcb chagne
pcb chagne
Parts:
- K01, K02, K03, K04, K05, K11, K12, K13, K14, K15, K21, K22, K23, K24, K25, K30, K31, K32: footprint keyswitches:SW_PG1350_reversible -> keyswitches:SW_MX_reversible
Connections:
- net k01: now also U1.37 (PB10)
- net k10: no longer names the net of U1.17 (PB9)
